Commit message: Initial URDF of Forth hand and Pisa hand
Signed-off-by: rnuti <r.nuti@hotmail.it>

File: forth_hand_description/model/forth_hand.urdf.xacro (robot description, xacro)
@@ -7,7 +7,7 @@
 	-->
 	<xacro:include filename="$(find forth_hand_description)/model/materials.urdf.xacro"/>
-	<xacro:include filename="$(find forth_hand_description)/model/forth_hand.transmission.xacro"/>
-	<xacro:include filename="$(find forth_hand_description)/model/forth_hand.gazebo.xacro"/>
-	<xacro:include filename="$(find forth_hand_description)/model/forth_hand.inertia.xacro"/>
+	<!-- <xacro:include filename="$(find forth_hand_description)/model/forth_hand.transmission.xacro"/> -->
+	<!--<xacro:include filename="$(find forth_hand_description)/model/forth_hand.gazebo.xacro"/>-->
+	<!-- <xacro:include filename="$(find forth_hand_description)/model/forth_hand.inertia.xacro"/> -->
 	<xacro:property name="pi" value="3.1415926535897931" />
 	<!-- joint properties -->
@@ -55,5 +55,5 @@
 	<!-- SOFT FINGER model -->
 	<!-- 4 fingers are equal (index, middle, ring, little) -->
-	<xacro:macro name="forth_finger" params="parent parent_name name position orientation useMimicTag abd_R ">
+	<xacro:macro name="forth_finger" params="parent parent_name name position orientation abd_R ">
 		<!-- KNUCKLE -->
 		<joint name="${name}_abd_joint" type="revolute">
@@ -64,7 +64,7 @@
 			<limit lower="${abd_lb *pi/180}" upper="${abd_ub *pi/180}" effort="${effort}" velocity="${velocity}"/>
 			<dynamics damping="${damping}" friction="${friction}"/>
-			<xacro:if value="${useMimicTag}">
+			<!-- <xacro:if value="${useMimicTag}">
 				<mimic joint="${parent_name}_synergy_joint" multiplier="${abd_R}"/>
-			</xacro:if>
+			</xacro:if> -->
 		</joint>
 		<link name="${name}_knuckle_link">
@@ -163,5 +163,5 @@
 	<!-- THUMB MODEL -->
 	<!-- It has one joint less than rest of fingers -->
-	<xacro:macro name="forth_thumb" params="parent parent_name name left position orientation useMimicTag abd_R ">
+	<xacro:macro name="forth_thumb" params="parent parent_name name left position orientation abd_R ">
 		 <xacro:if value="${left}">
 			<!-- KNUCKLE -->
@@ -173,7 +173,7 @@
 				<limit lower="${thumb_abd_lb *pi/180}" upper="${thumb_abd_ub *pi/180}" effort="${effort}" velocity="${velocity}"/>
 				<dynamics damping="${damping}" friction="${friction}"/>
-				<xacro:if value="${useMimicTag}">
+				<!-- <xacro:if value="${useMimicTag}">
 					<mimic joint="${parent_name}_synergy_joint" multiplier="${abd_R}"/>
-				</xacro:if>
+				</xacro:if> -->
 			</joint>
 			<link name="${name}_fake_link">
@@ -200,7 +200,7 @@
 				<limit lower="${thumb_abd_lb *pi/180}" upper="${thumb_abd_ub *pi/180}" effort="${effort}" velocity="${velocity}"/>
 				<dynamics damping="${damping}" friction="${friction}"/>
-				<xacro:if value="${useMimicTag}">
+				<!-- <xacro:if value="${useMimicTag}">
 					<mimic joint="${parent_name}_synergy_joint" multiplier="${abd_R}"/>
-				</xacro:if>
+				</xacro:if> -->
 			</joint>
 			<link name="${name}_knuckle_link">
@@ -240,7 +240,7 @@
 				<limit lower="${thumb_abd_lb *pi/180}" upper="${thumb_abd_ub *pi/180}" effort="${effort}" velocity="${velocity}"/>
 				<dynamics damping="${damping}" friction="${friction}"/>
-				<xacro:if value="${useMimicTag}">
+				<!-- <xacro:if value="${useMimicTag}">
 					<mimic joint="${parent_name}_synergy_joint" multiplier="${abd_R}"/>
-				</xacro:if>
+				</xacro:if> -->
 			</joint>
 			<link name="${name}_fake_link">
@@ -268,7 +268,7 @@
 				<limit lower="${thumb_abd_lb *pi/180}" upper="${thumb_abd_ub *pi/180}" effort="${effort}" velocity="${velocity}"/>
 				<dynamics damping="${damping}" friction="${friction}"/>
-				<xacro:if value="${useMimicTag}">
+				<!-- <xacro:if value="${useMimicTag}">
 					<mimic joint="${parent_name}_synergy_joint" multiplier="${abd_R}"/>
-				</xacro:if>
+				</xacro:if> -->
 			</joint>
 			<link name="${name}_knuckle_link">
@@ -341,5 +341,5 @@
 	</xacro:macro>
 	<!-- SOFT HAND MODEL -->
-	<xacro:macro name="forth_hand" params="parent name withAdaptiveTransmission useMimicTag left *origin">
+	<xacro:macro name="forth_hand" params="parent name  left *origin">
 		<!-- MOTOR JOINT -->
 <!--		<joint name="${name}_synergy_joint" type="revolute" >
@@ -397,20 +397,20 @@
 		<!-- change anchor points accordingly to the leftness -->
 		<xacro:if value="${left}">
-			<xacro:forth_thumb parent="${name}_palm_link" parent_name="${name}" name="${name}_thumb" left="${left}" position="0.005669722 -0.032876873 0.018373996" orientation="0.0 -0.43633198577877463 -1.570796326794897" useMimicTag="${useMimicTag}" abd_R="${thumb_abd_R *(thumb_abd_ub - thumb_abd_lb)*pi/180}" />
-			<xacro:forth_finger parent="${name}_palm_link" parent_name="${name}" name="${name}_index" position="-0.003349856 -0.019500000 0.058891802" orientation="-1.5707963267948957 -1.2217307407768807 -1.570796326794897" useMimicTag="${useMimicTag}" abd_R="${index_abd_R}" />
-			<xacro:forth_finger parent="${name}_palm_link" parent_name="${name}" name="${name}_middle" position="-0.003349856 0.0 0.072391802" orientation="-3.141592653589793 -1.5707963267948966 0.0" useMimicTag="${useMimicTag}" abd_R="${middle_abd_R}"  />
-			<xacro:forth_finger parent="${name}_palm_link" parent_name="${name}" name="${name}_ring" position="-0.003349856 0.019500000 0.058891802" orientation="1.5707963267948952 -1.3962636194521678 1.5707963267948966" useMimicTag="${useMimicTag}" abd_R="${ring_abd_R}"  />
-			<xacro:forth_finger parent="${name}_palm_link" parent_name="${name}" name="${name}_little" position="-0.00349856 0.039000000 0.045391802" orientation="1.5707963267948957 -1.2217307407768807 1.570796326794897" useMimicTag="${useMimicTag}" abd_R="${little_abd_R}"  />
+			<xacro:forth_thumb parent="${name}_palm_link" parent_name="${name}" name="${name}_thumb" left="${left}" position="0.005669722 -0.032876873 0.018373996" orientation="0.0 -0.43633198577877463 -1.570796326794897" abd_R="${thumb_abd_R *(thumb_abd_ub - thumb_abd_lb)*pi/180}" />
+			<xacro:forth_finger parent="${name}_palm_link" parent_name="${name}" name="${name}_index" position="-0.003349856 -0.019500000 0.058891802" orientation="-1.5707963267948957 -1.2217307407768807 -1.570796326794897" abd_R="${index_abd_R}" />
+			<xacro:forth_finger parent="${name}_palm_link" parent_name="${name}" name="${name}_middle" position="-0.003349856 0.0 0.072391802" orientation="-3.141592653589793 -1.5707963267948966 0.0" abd_R="${middle_abd_R}"  />
+			<xacro:forth_finger parent="${name}_palm_link" parent_name="${name}" name="${name}_ring" position="-0.003349856 0.019500000 0.058891802" orientation="1.5707963267948952 -1.3962636194521678 1.5707963267948966" abd_R="${ring_abd_R}"  />
+			<xacro:forth_finger parent="${name}_palm_link" parent_name="${name}" name="${name}_little" position="-0.00349856 0.039000000 0.045391802" orientation="1.5707963267948957 -1.2217307407768807 1.570796326794897" abd_R="${little_abd_R}"  />
 		</xacro:if>
 		<xacro:unless value="${left}">
 			<!-- <xacro:forth_thumb parent="${name}_palm_link" parent_name="${name}" name="${name}_thumb" left="${left}" position="0.005669722 0.032876873 0.018373996" orientation="0.08389097788000696 -0.4287012609015684 1.3712034099005517" useMimicTag="${useMimicTag}" abd_R="${thumb_abd_R *(thumb_abd_ub - thumb_abd_lb)*pi/180}"  /> -->
-			<xacro:forth_thumb parent="${name}_palm_link" parent_name="${name}" name="${name}_thumb" left="${left}" position="0.007 0.045 -0.045" orientation="0 0.41 1.57" useMimicTag="${useMimicTag}" abd_R="${thumb_abd_R *(thumb_abd_ub - thumb_abd_lb)*pi/180}"  />
-			<xacro:forth_finger parent="${name}_palm_link" parent_name="${name}" name="${name}_index" position="0.008 0.033 0.054" orientation="0 0 0" useMimicTag="${useMimicTag}" abd_R="${index_abd_R}"  />
-			<xacro:forth_finger parent="${name}_palm_link" parent_name="${name}" name="${name}_middle" position="0.008 0.010 0.062" orientation="0 0 0.0" useMimicTag="${useMimicTag}" abd_R="${middle_abd_R}"  />
-			<xacro:forth_finger parent="${name}_palm_link" parent_name="${name}" name="${name}_ring" position="0.008 -0.014 0.060" orientation="0 0 0" useMimicTag="${useMimicTag}" abd_R="${ring_abd_R}" />
-			<xacro:forth_finger parent="${name}_palm_link" parent_name="${name}" name="${name}_little" position=" 0.008 -0.034 0.051" orientation="0 0 0" useMimicTag="${useMimicTag}" abd_R="${little_abd_R}" />
+			<xacro:forth_thumb parent="${name}_palm_link" parent_name="${name}" name="${name}_thumb" left="${left}" position="0.007 0.045 -0.045" orientation="0 0.41 1.57"  abd_R="${thumb_abd_R *(thumb_abd_ub - thumb_abd_lb)*pi/180}"  />
+			<xacro:forth_finger parent="${name}_palm_link" parent_name="${name}" name="${name}_index" position="0.008 0.033 0.054" orientation="0 0 0" abd_R="${index_abd_R}"  />
+			<xacro:forth_finger parent="${name}_palm_link" parent_name="${name}" name="${name}_middle" position="0.008 0.010 0.062" orientation="0 0 0.0" abd_R="${middle_abd_R}"  />
+			<xacro:forth_finger parent="${name}_palm_link" parent_name="${name}" name="${name}_ring" position="0.008 -0.014 0.060" orientation="0 0 0"  abd_R="${ring_abd_R}" />
+			<xacro:forth_finger parent="${name}_palm_link" parent_name="${name}" name="${name}_little" position=" 0.008 -0.034 0.051" orientation="0 0 0" abd_R="${little_abd_R}" />
 		</xacro:unless>
-		<xacro:forth_hand_transmission name="${name}" withAdaptiveTransmission="${withAdaptiveTransmission}"/>
-		<xacro:forth_hand_gazebo name="${name}" withAdaptiveTransmission="${withAdaptiveTransmission}" useMimicTag="${useMimicTag}"/>
+		<!-- <xacro:forth_hand_transmission name="${name}" withAdaptiveTransmission="${withAdaptiveTransmission}"/>
+		<xacro:forth_hand_gazebo name="${name}" withAdaptiveTransmission="${withAdaptiveTransmission}" useMimicTag="${useMimicTag}"/> -->
 	</xacro:macro>
 </robot>

File: forth_hand_description/robot/forth_hand_simple.urdf.xacro (robot description, xacro)
@@ -3,8 +3,8 @@
 	<xacro:include filename="$(find forth_hand_description)/model/forth_hand.urdf.xacro"/>
 	<link name="box">
-		<inertial>
+	<!-- 	<inertial>
 			<mass value="50.0"/>
 			<inertia  ixx="1" ixy="0.00"  ixz="0.00" iyy="1" iyz="0.00" izz="1" />
-		</inertial>
+		</inertial> -->
 		<visual>
 			<origin xyz="0 0 0.50" rpy="0 0 0"/>
@@ -13,10 +13,10 @@
 			</geometry>
 		</visual>
-		<collision>
+		<!-- <collision>
 			<origin xyz="0 0 0.50" rpy="0 0 0"/>
 			<geometry>
 				<box size="1.0 1.0 1.0"/>
 			</geometry>
-		</collision>
+		</collision> -->
 	</link>
 <!--
@@ -76,21 +76,21 @@
 	</joint>
 	<link name="wrist_right">
-		<inertial>
+		<!--<inertial>
 			<mass value="1.0"/>
 			<inertia  ixx="0.01" ixy="0.00"  ixz="0.00" iyy="0.01" iyz="0.00" izz="0.01" />
-		</inertial>
-		<visual>
+		</inertial>-->
+		<!--<visual>
 			<geometry>
 				<mesh filename="package://forth_hand_description/meshes/coman_coupler_right.stl" scale=" .001 .001 .001" />
 			</geometry>
 			<material name="SoftHand/LightBlue" />
-		</visual>
-		<collision>
-			<geometry>
+		</visual>-->
+		<!--<collision>
+			 <geometry>
 				<mesh filename="package://forth_hand_description/meshes/coman_coupler_right.stl" scale=" .001 .001 .001" />
 			</geometry>
-		</collision>
+		</collision>-->
 	</link>
-	<xacro:forth_hand parent="wrist_right" name="forth_hand_right" withAdaptiveTransmission="false" useMimicTag="$(arg use_mimic_tag)" left="false">
+	<xacro:forth_hand parent="wrist_right" name="forth_hand_right" left="false">
 		<origin xyz="0.002 0.009 0.038" rpy="0 0 0"/>
 	</xacro:forth_hand>

File: pisa_hand_description/model/pisa_hand.urdf.xacro (robot description, xacro)
@@ -7,7 +7,7 @@
 	-->
 	<xacro:include filename="$(find pisa_hand_description)/model/materials.urdf.xacro"/>
-	<xacro:include filename="$(find pisa_hand_description)/model/pisa_hand.transmission.xacro"/>
-	<xacro:include filename="$(find pisa_hand_description)/model/pisa_hand.gazebo.xacro"/>
-	<xacro:include filename="$(find pisa_hand_description)/model/pisa_hand.inertia.xacro"/>
+	<!-- <xacro:include filename="$(find pisa_hand_description)/model/pisa_hand.transmission.xacro"/> -->
+	<!-- <xacro:include filename="$(find pisa_hand_description)/model/pisa_hand.gazebo.xacro"/> -->
+	<!-- <xacro:include filename="$(find pisa_hand_description)/model/pisa_hand.inertia.xacro"/> -->
 	<xacro:property name="pi" value="3.1415926535897931" />
 	<!-- joint properties -->
@@ -55,5 +55,5 @@
 	<!-- SOFT FINGER model -->
 	<!-- 4 fingers are equal (index, middle, ring, little) -->
-	<xacro:macro name="soft_finger" params="parent parent_name name position orientation useMimicTag abd_R ">
+	<xacro:macro name="soft_finger" params="parent parent_name name position orientation abd_R ">
 		<!-- KNUCKLE -->
 		<joint name="${name}_abd_joint" type="revolute">
@@ -64,7 +64,7 @@
 			<limit lower="${abd_lb *pi/180}" upper="${abd_ub *pi/180}" effort="${effort}" velocity="${velocity}"/>
 			<dynamics damping="${damping}" friction="${friction}"/>
-			<xacro:if value="${useMimicTag}">
+			<!-- <xacro:if value="${useMimicTag}">
 				<mimic joint="${parent_name}_synergy_joint" multiplier="${abd_R}"/>
-			</xacro:if>
+			</xacro:if> -->
 		</joint>
 		<link name="${name}_knuckle_link">
@@ -163,5 +163,5 @@
 	<!-- THUMB MODEL -->
 	<!-- It has one joint less than rest of fingers -->
-	<xacro:macro name="soft_thumb" params="parent parent_name name left position orientation useMimicTag abd_R ">
+	<xacro:macro name="soft_thumb" params="parent parent_name name left position orientation abd_R ">
 		 <xacro:if value="${left}">
 			<!-- KNUCKLE -->
@@ -173,7 +173,7 @@
 				<limit lower="${thumb_abd_lb *pi/180}" upper="${thumb_abd_ub *pi/180}" effort="${effort}" velocity="${velocity}"/>
 				<dynamics damping="${damping}" friction="${friction}"/>
-				<xacro:if value="${useMimicTag}">
+				<!-- <xacro:if value="${useMimicTag}">
 					<mimic joint="${parent_name}_synergy_joint" multiplier="${abd_R}"/>
-				</xacro:if>
+				</xacro:if> -->
 			</joint>
 			<link name="${name}_fake_link">
@@ -200,7 +200,7 @@
 				<limit lower="${thumb_abd_lb *pi/180}" upper="${thumb_abd_ub *pi/180}" effort="${effort}" velocity="${velocity}"/>
 				<dynamics damping="${damping}" friction="${friction}"/>
-				<xacro:if value="${useMimicTag}">
+				<!-- <xacro:if value="${useMimicTag}">
 					<mimic joint="${parent_name}_synergy_joint" multiplier="${abd_R}"/>
-				</xacro:if>
+				</xacro:if> -->
 			</joint>
 			<link name="${name}_knuckle_link">
@@ -240,7 +240,7 @@
 				<limit lower="${thumb_abd_lb *pi/180}" upper="${thumb_abd_ub *pi/180}" effort="${effort}" velocity="${velocity}"/>
 				<dynamics damping="${damping}" friction="${friction}"/>
-				<xacro:if value="${useMimicTag}">
+				<!-- <xacro:if value="${useMimicTag}">
 					<mimic joint="${parent_name}_synergy_joint" multiplier="${abd_R}"/>
-				</xacro:if>
+				</xacro:if> -->
 			</joint>
 			<link name="${name}_fake_link">
@@ -268,7 +268,7 @@
 				<limit lower="${thumb_abd_lb *pi/180}" upper="${thumb_abd_ub *pi/180}" effort="${effort}" velocity="${velocity}"/>
 				<dynamics damping="${damping}" friction="${friction}"/>
-				<xacro:if value="${useMimicTag}">
+				<!-- <xacro:if value="${useMimicTag}">
 					<mimic joint="${parent_name}_synergy_joint" multiplier="${abd_R}"/>
-				</xacro:if>
+				</xacro:if> -->
 			</joint>
 			<link name="${name}_knuckle_link">
@@ -341,5 +341,5 @@
 	</xacro:macro>
 	<!-- SOFT HAND MODEL -->
-	<xacro:macro name="pisa_hand" params="parent name withAdaptiveTransmission useMimicTag left *origin">
+	<xacro:macro name="pisa_hand" params="parent name left *origin">
 		<!-- MOTOR JOINT -->
 	<!--	<joint name="${name}_synergy_joint" type="revolute" >
@@ -396,20 +396,20 @@
 		<!-- change anchor points accordingly to the leftness -->
 		<xacro:if value="${left}">
-			<xacro:soft_thumb parent="${name}_palm_link" parent_name="${name}" name="${name}_thumb" left="${left}" position="0.005669722 -0.032876873 0.018373996" orientation="0.0 -0.43633198577877463 -1.570796326794897" useMimicTag="${useMimicTag}" abd_R="${thumb_abd_R *(thumb_abd_ub - thumb_abd_lb)*pi/180}" />
-			<xacro:soft_finger parent="${name}_palm_link" parent_name="${name}" name="${name}_index" position="-0.003349856 -0.019500000 0.058891802" orientation="-1.5707963267948957 -1.2217307407768807 -1.570796326794897" useMimicTag="${useMimicTag}" abd_R="${index_abd_R}" />
-			<xacro:soft_finger parent="${name}_palm_link" parent_name="${name}" name="${name}_middle" position="-0.003349856 0.0 0.072391802" orientation="-3.141592653589793 -1.5707963267948966 0.0" useMimicTag="${useMimicTag}" abd_R="${middle_abd_R}"  />
-			<xacro:soft_finger parent="${name}_palm_link" parent_name="${name}" name="${name}_ring" position="-0.003349856 0.019500000 0.058891802" orientation="1.5707963267948952 -1.3962636194521678 1.5707963267948966" useMimicTag="${useMimicTag}" abd_R="${ring_abd_R}"  />
-			<xacro:soft_finger parent="${name}_palm_link" parent_name="${name}" name="${name}_little" position="-0.00349856 0.039000000 0.045391802" orientation="1.5707963267948957 -1.2217307407768807 1.570796326794897" useMimicTag="${useMimicTag}" abd_R="${little_abd_R}"  />
+			<xacro:soft_thumb parent="${name}_palm_link" parent_name="${name}" name="${name}_thumb" left="${left}" position="0.005669722 -0.032876873 0.018373996" orientation="0.0 -0.43633198577877463 -1.570796326794897"  abd_R="${thumb_abd_R *(thumb_abd_ub - thumb_abd_lb)*pi/180}" />
+			<xacro:soft_finger parent="${name}_palm_link" parent_name="${name}" name="${name}_index" position="-0.003349856 -0.019500000 0.058891802" orientation="-1.5707963267948957 -1.2217307407768807 -1.570796326794897" abd_R="${index_abd_R}" />
+			<xacro:soft_finger parent="${name}_palm_link" parent_name="${name}" name="${name}_middle" position="-0.003349856 0.0 0.072391802" orientation="-3.141592653589793 -1.5707963267948966 0.0" abd_R="${middle_abd_R}"  />
+			<xacro:soft_finger parent="${name}_palm_link" parent_name="${name}" name="${name}_ring" position="-0.003349856 0.019500000 0.058891802" orientation="1.5707963267948952 -1.3962636194521678 1.5707963267948966"  abd_R="${ring_abd_R}"  />
+			<xacro:soft_finger parent="${name}_palm_link" parent_name="${name}" name="${name}_little" position="-0.00349856 0.039000000 0.045391802" orientation="1.5707963267948957 -1.2217307407768807 1.570796326794897"  abd_R="${little_abd_R}"  />
 		</xacro:if>
 		<xacro:unless value="${left}">
 			<!-- <xacro:soft_thumb parent="${name}_palm_link" parent_name="${name}" name="${name}_thumb" left="${left}" position="0.005669722 0.032876873 0.018373996" orientation="0.08389097788000696 -0.4287012609015684 1.3712034099005517" useMimicTag="${useMimicTag}" abd_R="${thumb_abd_R *(thumb_abd_ub - thumb_abd_lb)*pi/180}"  /> -->
-			<xacro:soft_thumb parent="${name}_palm_link" parent_name="${name}" name="${name}_thumb" left="${left}" position="0.007 0.045 -0.045" orientation="0 -1.16 1.57" useMimicTag="${useMimicTag}" abd_R="${thumb_abd_R *(thumb_abd_ub - thumb_abd_lb)*pi/180}"  />
-			<xacro:soft_finger parent="${name}_palm_link" parent_name="${name}" name="${name}_index" position="0.008 0.033 0.054" orientation="0 0 0" useMimicTag="${useMimicTag}" abd_R="${index_abd_R}"  />
-			<xacro:soft_finger parent="${name}_palm_link" parent_name="${name}" name="${name}_middle" position="0.008 0.010 0.062" orientation="0 0 0.0" useMimicTag="${useMimicTag}" abd_R="${middle_abd_R}"  />
-			<xacro:soft_finger parent="${name}_palm_link" parent_name="${name}" name="${name}_ring" position="0.008 -0.014 0.060" orientation="0 0 0" useMimicTag="${useMimicTag}" abd_R="${ring_abd_R}" />
-			<xacro:soft_finger parent="${name}_palm_link" parent_name="${name}" name="${name}_little" position=" 0.008 -0.034 0.051" orientation="0 0 0" useMimicTag="${useMimicTag}" abd_R="${little_abd_R}" />
+			<xacro:soft_thumb parent="${name}_palm_link" parent_name="${name}" name="${name}_thumb" left="${left}" position="0.007 0.045 -0.045" orientation="0 -1.16 1.57" abd_R="${thumb_abd_R *(thumb_abd_ub - thumb_abd_lb)*pi/180}"  />
+			<xacro:soft_finger parent="${name}_palm_link" parent_name="${name}" name="${name}_index" position="0.008 0.033 0.054" orientation="0 0 0"  abd_R="${index_abd_R}"  />
+			<xacro:soft_finger parent="${name}_palm_link" parent_name="${name}" name="${name}_middle" position="0.008 0.010 0.062" orientation="0 0 0.0" abd_R="${middle_abd_R}"  />
+			<xacro:soft_finger parent="${name}_palm_link" parent_name="${name}" name="${name}_ring" position="0.008 -0.014 0.060" orientation="0 0 0" abd_R="${ring_abd_R}" />
+			<xacro:soft_finger parent="${name}_palm_link" parent_name="${name}" name="${name}_little" position=" 0.008 -0.034 0.051" orientation="0 0 0" abd_R="${little_abd_R}" />
 		</xacro:unless>
-		<xacro:pisa_hand_transmission name="${name}" withAdaptiveTransmission="${withAdaptiveTransmission}"/>
-		<xacro:pisa_hand_gazebo name="${name}" withAdaptiveTransmission="${withAdaptiveTransmission}" useMimicTag="${useMimicTag}"/>
+		<!-- <xacro:pisa_hand_transmission name="${name}" withAdaptiveTransmission="${withAdaptiveTransmission}"/>
+		<xacro:pisa_hand_gazebo name="${name}" withAdaptiveTransmission="${withAdaptiveTransmission}" useMimicTag="${useMimicTag}"/> -->
 	</xacro:macro>
 </robot>

File: pisa_hand_description/robot/pisa_hand_simple.urdf.xacro (robot description, xacro)
@@ -3,8 +3,8 @@
 	<xacro:include filename="$(find pisa_hand_description)/model/pisa_hand.urdf.xacro"/>
 	<link name="box">
-		<inertial>
+		<!-- <inertial>
 			<mass value="50.0"/>
 			<inertia  ixx="1" ixy="0.00"  ixz="0.00" iyy="1" iyz="0.00" izz="1" />
-		</inertial>
+		</inertial> -->
 		<visual>
 			<origin xyz="0 0 0.50" rpy="0 0 0"/>
@@ -13,10 +13,10 @@
 			</geometry>
 		</visual>
-		<collision>
+		<!-- <collision>
 			<origin xyz="0 0 0.50" rpy="0 0 0"/>
 			<geometry>
 				<box size="1.0 1.0 1.0"/>
 			</geometry>
-		</collision>
+		</collision> -->
 	</link>
 <!--
@@ -76,5 +76,5 @@
 	</joint>
 	<link name="wrist_right">
-		<inertial>
+		<!-- <inertial>
 			<mass value="1.0"/>
 			<inertia  ixx="0.01" ixy="0.00"  ixz="0.00" iyy="0.01" iyz="0.00" izz="0.01" />
@@ -90,7 +90,7 @@
 				<mesh filename="package://pisa_hand_description/meshes/coman_coupler_right.stl" scale=" .001 .001 .001" />
 			</geometry>
-		</collision>
+		</collision> -->
 	</link>
-	<xacro:pisa_hand parent="wrist_right" name="pisa_hand_right" withAdaptiveTransmission="true" useMimicTag="$(arg use_mimic_tag)" left="false">
+	<xacro:pisa_hand parent="wrist_right" name="pisa_hand_right" left="false">
 		<origin xyz="0.002 0.009 0.038" rpy="0 0 0"/>
 	</xacro:pisa_hand>
